Commit message: Some updates

File: description/camera.xacro (robot description, xacro)
@@ -3,8 +3,8 @@
     <joint name="camera_joint" type="fixed">
         <parent link="base"/>
-        <child link="camera_link"/>
+        <child link="camera"/>
         <origin xyz="-0.14 0.0 0.10" rpy="0 0 ${pi}"/>
     </joint>
-    <link name="camera_link">
+    <link name="camera">
         <visual>
             <geometry>
@@ -15,11 +15,11 @@
     </link>
     <joint name="camera_optical_joint" type="fixed">
-        <parent link="camera_link"/>
-        <child link="camera_link_optical"/>
+        <parent link="camera"/>
+        <child link="camera_optical"/>
         <origin xyz="0 0 0" rpy="${-pi/2} 0 ${-pi/2}"/>
     </joint>
-    <link name="camera_link_optical">
+    <link name="camera_optical">
     </link>
-    <gazebo reference="camera_link">
+    <gazebo reference="camera">
         <material>Gazebo/Black</material>
         <sensor name="camera" type="camera">
@@ -41,6 +41,6 @@
             <plugin name="camera_controller" filename="libgazebo_ros_camera.so">
                 <ros>
-                <namespace>KapiBara</namespace>
-                <remapping>~/out:=camera</remapping>
+                    <namespace>KapiBara</namespace>
+                    <remapping>~/out:=camera</remapping>
                 </ros>
                 <frame_name>camera_link_optical</frame_name>

File: description/lasers_def.xacro (robot description, xacro)
@@ -37,8 +37,8 @@
             <plugin name="${sensor_name}_laserscan" filename="libgazebo_ros_ray_sensor.so">
                 <ros>
-                <namespace>Gazebo</namespace>
-                <remapping>~/out:=${sensor_name}</remapping>
+                    <namespace>KapiBara</namespace>
+                    <remapping>~/out:=${sensor_name}</remapping>
                 </ros>
-                <output_type>sensor_msgs/Range</output_type>
+                <output_type>sensor_msgs/LaserScan</output_type>
                 <radiation_type>infrared</radiation_type>
                 <frame_name>${sensor_name}_laser</frame_name>

File: description/lasers_joints.xacro (robot description, xacro)
@@ -22,18 +22,4 @@
     </joint>
     <link name="front_right_laser_link">
-        <visual>
-            <geometry>
-                <box size="0.01 0.01 0.01" />
-            </geometry>
-            <material name="red" />
-        </visual>
-    </link>
-    <!-- FLOOR DISTANCE SENSOR -->
-    <joint name="floor_laser_joint" type="fixed">
-        <parent link="base"/>
-        <child link="floor_laser_link"/>
-        <origin xyz="-0.16 0.0 0.021" rpy="0 ${pi/5} ${pi}"/>
-    </joint>
-    <link name="floor_laser_link">
         <visual>
             <geometry>

File: description/robot_core.xacro (robot description, xacro)
@@ -1,4 +1,4 @@
 <?xml version="1.0"?>
-<robot xmlns:xacro="http://www.ros.org/wiki/xacro" name="robot">
+<robot xmlns:xacro="http://www.ros.org/wiki/xacro" name="kapibara_robot">
     <xacro:include filename="inertial_macros.xacro"/>
     <material name="white">
@@ -31,13 +31,4 @@
             <material name="black" />
         </visual>
-        <collision>
-            <origin xyz="0 0 0.02" />
-            <geometry>
-                <box size="0.150 0.083 0.033" />
-            </geometry>
-        </collision>
-        <xacro:inertial_box mass="0.65" x="0.15" y="0.083" z="0.033" >
-            <origin xyz="0 0 0.02" rpy="0 0 0" />
-        </xacro:inertial_box>
     </link>
     <gazebo reference="chassis">
@@ -58,5 +49,5 @@
             <material name="orange" />
         </visual>
-        <collision>
+        <collision name="base_collision">
             <origin xyz="-0.02 0 0.07" />
             <geometry>
@@ -70,4 +61,18 @@
     <gazebo reference="base">
         <material>Gazebo/Orange</material>
+        <sensor type="contact" name="contact_sensor">
+            <always_on>true</always_on>
+            <update_rate>50</update_rate>
+            <contact>
+            <collision>base_link_fixed_joint_lump__base_collision_collision</collision>
+            </contact>
+            <plugin name="bumper_plugin_kapibara" filename="libgazebo_ros_bumper.so">
+                <alwaysOn>true</alwaysOn>
+                <frameName>base</frameName>
+                <ros>
+                <remapping>bumper_states:=collision</remapping>
+                </ros>
+            </plugin>
+      </sensor>
     </gazebo>
     <!-- LEFT WHEEL LINK -->
@@ -76,5 +81,7 @@
         <child link="left_wheel1" />
         <axis xyz="0 0 1"/>
-        <origin rpy="${-pi/2} 0 0" xyz="0.065 0.066 0.0165"/>
+        <origin rpy="${-pi/2} 0 0" xyz="0.005 0.066 0.0135"/>
+        <!-- <joint_properties damping="1.0" friction="1.0" />  -->
+        <!-- <limit effort="10000" velocity="1000"/>  -->
     </joint>
     <link name="left_wheel1">
@@ -93,12 +100,17 @@
         </collision>
         <xacro:inertial_cylinder mass="0.1" radius="0.024" length="0.044">
-            <origin xyz="0 0 0" rpy="0 0 1" />
-        </xacro:inertial_cylinder>
-    </link>
+            <origin xyz="0 0 0" rpy="0 0 0" />
+        </xacro:inertial_cylinder>
+    </link>
+    <gazebo reference="left_wheel1">
+        <material>Gazebo/White</material>
+        <mu1 value="0.5"/>
+        <mu2 value="0.5"/>
+    </gazebo>
     <joint name="wheel_left2_joint" type="continuous">
         <parent link="chassis" />
         <child link="left_wheel2" />
         <axis xyz="0 0 1"/>
-        <origin rpy="${-pi/2} 0 0" xyz="0.005 0.066 0.0165"/>
+        <origin rpy="${-pi/2} 0 0" xyz="0.065 0.066 0.0135"/>
     </joint>
     <link name="left_wheel2">
@@ -117,12 +129,17 @@
         </collision>
         <xacro:inertial_cylinder mass="0.1" radius="0.024" length="0.044">
-            <origin xyz="0 0 0" rpy="0 0 1" />
-        </xacro:inertial_cylinder>
-    </link>
+            <origin xyz="0 0 0" rpy="0 0 0" />
+        </xacro:inertial_cylinder>
+    </link>
+    <gazebo reference="left_wheel2">
+        <material>Gazebo/White</material>
+        <mu1 value="0.5"/>
+        <mu2 value="0.5"/>
+    </gazebo>
     <joint name="wheel_left3_joint" type="continuous">
         <parent link="chassis" />
         <child link="left_wheel3" />
         <axis xyz="0 0 1"/>
-        <origin rpy="${-pi/2} 0 0" xyz="-0.055 0.066 0.0165"/>
+        <origin rpy="${-pi/2} 0 0" xyz="-0.055 0.066 0.0135"/>
     </joint>
     <link name="left_wheel3">
@@ -141,7 +158,12 @@
         </collision>
         <xacro:inertial_cylinder mass="0.1" radius="0.024" length="0.044">
-            <origin xyz="0 0 0" rpy="0 0 1" />
-        </xacro:inertial_cylinder>
-    </link>
+            <origin xyz="0 0 0" rpy="0 0 0" />
+        </xacro:inertial_cylinder>
+    </link>
+    <gazebo reference="left_wheel3">
+        <material>Gazebo/White</material>
+        <mu1 value="0.5"/>
+        <mu2 value="0.5"/>
+    </gazebo>
     <!-- RIGHT WHEEL LINK -->
     <joint name="wheel_right1_joint" type="continuous">
@@ -149,5 +171,7 @@
         <child link="right_wheel1" />
         <axis xyz="0 0 1"/>
-        <origin rpy="${-pi/2} 0 0" xyz="0.065 -0.066 0.0165"/>
+        <origin rpy="${-pi/2} 0 0" xyz="0.005 -0.066 0.0135"/>
+        <!-- <joint_properties damping="1.0" friction="1.0" />  -->
+        <!-- <limit effort="10000" velocity="1000"/>  -->
     </joint>
     <link name="right_wheel1">
@@ -166,12 +190,17 @@
         </collision>
         <xacro:inertial_cylinder mass="0.1" radius="0.024" length="0.044">
-            <origin xyz="0 0 0" rpy="0 0 1" />
-        </xacro:inertial_cylinder>
-    </link>
+            <origin xyz="0 0 0" rpy="0 0 0" />
+        </xacro:inertial_cylinder>
+    </link>
+    <gazebo reference="right_wheel1">
+        <material>Gazebo/White</material>
+        <mu1 value="0.5"/>
+        <mu2 value="0.5"/>
+    </gazebo>
     <joint name="wheel_right2_joint" type="continuous">
         <parent link="chassis" />
         <child link="right_wheel2" />
         <axis xyz="0 0 1"/>
-        <origin rpy="${-pi/2} 0 0" xyz="0.005 -0.066 0.0165"/>
+        <origin rpy="${-pi/2} 0 0" xyz="0.065 -0.066 0.0135"/>
     </joint>
     <link name="right_wheel2">
@@ -190,12 +219,17 @@
         </collision>
         <xacro:inertial_cylinder mass="0.1" radius="0.024" length="0.044">
-            <origin xyz="0 0 0" rpy="0 0 1" />
-        </xacro:inertial_cylinder>
-    </link>
+            <origin xyz="0 0 0" rpy="0 0 0" />
+        </xacro:inertial_cylinder>
+    </link>
+    <gazebo reference="right_wheel2">
+        <material>Gazebo/White</material>
+        <mu1 value="0.5"/>
+        <mu2 value="0.5"/>
+    </gazebo>
     <joint name="wheel_right3_joint" type="continuous">
         <parent link="chassis" />
         <child link="right_wheel3" />
         <axis xyz="0 0 1"/>
-        <origin rpy="${-pi/2} 0 0" xyz="-0.055 -0.066 0.0165"/>
+        <origin rpy="${-pi/2} 0 0" xyz="-0.055 -0.066 0.0135"/>
     </joint>
     <link name="right_wheel3">
@@ -214,13 +248,18 @@
         </collision>
         <xacro:inertial_cylinder mass="0.1" radius="0.024" length="0.044">
-            <origin xyz="0 0 0" rpy="0 0 1" />
-        </xacro:inertial_cylinder>
-    </link>
+            <origin xyz="0 0 0" rpy="0 0 0" />
+        </xacro:inertial_cylinder>
+    </link>
+    <gazebo reference="right_wheel3">
+        <material>Gazebo/White</material>
+        <mu1 value="0.5"/>
+        <mu2 value="0.5"/>
+    </gazebo>
     <!-- EARS -->
     <joint name="left_ear_joint" type="revolute">
         <parent link="base" />
         <child link="left_ear" />
-        <axis xyz="0 1 0"/>
-        <origin rpy="0 ${-pi/2} 0" xyz="-0.09 0.075 0.09" />
+        <axis xyz="0 -1 0"/>
+        <origin rpy="0 ${pi/2} 0" xyz="-0.09 0.075 0.09" />
         <limit effort="1" velocity="1" upper="${pi}" lower="0" />
     </joint>
@@ -246,6 +285,6 @@
         <parent link="base" />
         <child link="righ_ear" />
-        <axis xyz="0 1 0"/>
-        <origin rpy="0 ${-pi/2} 0" xyz="-0.09 -0.070 0.09" />
+        <axis xyz="0 -1 0"/>
+        <origin rpy="0 ${pi/2} 0" xyz="-0.09 -0.070 0.09" />
         <limit effort="1" velocity="1" upper="${pi}" lower="0" />
     </joint>

File: description/ros2_control.xacro (robot description, xacro)
@@ -4,13 +4,11 @@
         <ros2_control name="KapiBaraMotors" type="system">
             <hardware>
-                <plugin>tb6612_drive_simple/TB6612DriveSimple</plugin>
+                <plugin>vel_saltis_drive/VelSaltisDrive</plugin>
                 <param name="left_wheel_name">wheel_left1_joint</param>
                 <param name="right_wheel_name">wheel_right3_joint</param>
+                <!-- <param name="left_ear">left_ear_joint</param>
+                <param name="right_ear">right_ear_joint</param> -->
                 <param name="max_speed">10</param>
                 <param name="loop_rate">30</param>
-                <param name="left_gpioA">406</param>
-                <param name="left_gpioB">407</param>
-                <param name="right_gpioA">404</param>
-                <param name="right_gpioB">405</param>
             </hardware>
             <joint name="wheel_left1_joint">
@@ -28,4 +26,40 @@
                 </command_interface>
                 <state_interface name="velocity" />
+                <state_interface name="position" />
+            </joint>
+            <!-- <joint name="right_ear_joint">
+                <command_interface name="position">
+                    <param name="min">-10</param>
+                    <param name="max">10</param>
+                </command_interface>
+                <state_interface name="position" />
+            </joint>
+            <joint name="left_ear_joint">
+                <command_interface name="position">
+                    <param name="min">-10</param>
+                    <param name="max">10</param>
+                </command_interface>
+                <state_interface name="position" />
+            </joint> -->
+        </ros2_control>
+        <ros2_control name="KapiBaraEars" type="system">
+            <hardware>
+                <plugin>vel_saltis_ears/VelSaltisEars</plugin>
+                <param name="left_ear_name">left_ear_joint</param>
+                <param name="right_ear_name">right_ear_joint</param>
+                <param name="loop_rate">30</param>
+            </hardware>
+            <joint name="right_ear_joint">
+                <command_interface name="position">
+                    <param name="min">-10</param>
+                    <param name="max">10</param>
+                </command_interface>
+                <state_interface name="position" />
+            </joint>
+            <joint name="left_ear_joint">
+                <command_interface name="position">
+                    <param name="min">-10</param>
+                    <param name="max">10</param>
+                </command_interface>
                 <state_interface name="position" />
             </joint>
@@ -53,8 +87,28 @@
                 <state_interface name="position" />
             </joint>
+            <joint name="right_ear_joint">
+                <command_interface name="position">
+                    <param name="min">-10</param>
+                    <param name="max">10</param>
+                </command_interface>
+                <state_interface name="position" />
+            </joint>
+            <joint name="left_ear_joint">
+                <command_interface name="position">
+                    <param name="min">-10</param>
+                    <param name="max">10</param>
+                </command_interface>
+                <state_interface name="position" />
+            </joint>
         </ros2_control>
     </xacro:if>
     <gazebo>
-        <plugin name="gazebo_ros2_control" filename="libgazebo_ros2_control.so">
+        <plugin name="kapibara_gazebo_ros2_control" filename="libgazebo_ros2_control.so">
+            <ros>
+                <namespace>KapiBara</namespace>
+                <remapping>/tf:=/KapiBara/tf</remapping>
+                <remapping>/tf_static:=/KapiBara/tf_static</remapping>
+            </ros>
+            <robot_param_node>/KapiBara/robot_state_publisher</robot_param_node>
             <parameters>$(find kapibara)/config/my_controllers.yaml</parameters>
             <parameters>$(find kapibara)/config/my_controllers_sim.yaml</parameters>
