Commit message: I have fixed problem with TF

File: description/camera.xacro (robot description, xacro)
@@ -1,10 +1,10 @@
 <?xml version="1.0"?>
 <robot xmlns:xacro="http://www.ros.org/wiki/xacro">
-    <joint name="camera_joint" type="fixed">
-        <parent link="base"/>
-        <child link="camera"/>
+    <joint name="/$(arg robot_name)/camera_joint" type="fixed">
+        <parent link="/$(arg robot_name)/base"/>
+        <child link="/$(arg robot_name)/camera"/>
         <origin xyz="-0.14 0.0 0.10" rpy="0 0 ${pi}"/>
     </joint>
-    <link name="camera">
+    <link name="/$(arg robot_name)/camera">
         <visual>
             <geometry>
@@ -14,14 +14,14 @@
         </visual>
     </link>
-    <joint name="camera_optical_joint" type="fixed">
-        <parent link="camera"/>
-        <child link="camera_optical"/>
+    <joint name="/$(arg robot_name)/camera_optical_joint" type="fixed">
+        <parent link="/$(arg robot_name)/camera"/>
+        <child link="/$(arg robot_name)/camera_optical"/>
         <origin xyz="0 0 0" rpy="${-pi/2} 0 ${-pi/2}"/>
     </joint>
-    <link name="camera_optical">
+    <link name="/$(arg robot_name)/camera_optical">
     </link>
-    <gazebo reference="camera">
+    <gazebo reference="/$(arg robot_name)/camera">
         <material>Gazebo/Black</material>
-        <sensor name="camera" type="camera">
+        <sensor name="kapibara_camera" type="camera">
             <pose> 0 0 0 0 0 0 </pose>
             <visualize>true</visualize>
@@ -41,8 +41,8 @@
             <plugin name="camera_controller" filename="libgazebo_ros_camera.so">
                 <ros>
-                    <namespace>KapiBara</namespace>
+                    <namespace>$(arg robot_name)</namespace>
                     <remapping>~/out:=camera</remapping>
                 </ros>
-                <frame_name>camera_link_optical</frame_name>
+                <frame_name>/$(arg robot_name)/camera_link_optical</frame_name>
             </plugin>
         </sensor>

File: description/imu.xacro (robot description, xacro)
@@ -1,12 +1,12 @@
 <?xml version="1.0"?>
 <robot xmlns:xacro="http://www.ros.org/wiki/xacro">
-    <joint name="imu_joint" type="fixed">
-        <parent link="chassis"/>
-        <child link="imu_link"/>
+    <joint name="/$(arg robot_name)/imu_joint" type="fixed">
+        <parent link="/$(arg robot_name)/chassis"/>
+        <child link="/$(arg robot_name)/imu_link"/>
         <origin xyz="0 0 0" rpy="0 0 0"/>
     </joint>
-    <link name="imu_link">
+    <link name="/$(arg robot_name)/imu_link">
     </link>
-    <gazebo reference="imu_link">
+    <gazebo reference="/$(arg robot_name)/imu_link">
     <sensor name="kapibara_imu" type="imu">
         <always_on>true</always_on>
@@ -56,5 +56,5 @@
         <plugin name="kapibara_imu" filename="libgazebo_ros_imu_sensor.so">
             <ros>
-                <namespace>KapiBara</namespace>
+                <namespace>$(arg robot_name)</namespace>
                 <remapping>~/out:=imu</remapping>
             </ros>

File: description/lasers_def.xacro (robot description, xacro)
@@ -2,7 +2,7 @@
 <robot xmlns:xacro="http://www.ros.org/wiki/xacro">
     <xacro:macro name="laser_sensor" params="sensor_name">
-    <gazebo reference="${sensor_name}_laser_link">
+    <gazebo reference="/$(arg robot_name)/${sensor_name}_laser_link">
         <material>Gazebo/Red</material>
-        <sensor name="${sensor_name}_laser" type="ray">
+        <sensor name="/$(arg robot_name)/${sensor_name}_laser" type="ray">
             <pose> 0 0 0 0 0 0 </pose>
             <always_on>true</always_on>
@@ -37,10 +37,10 @@
             <plugin name="${sensor_name}_laserscan" filename="libgazebo_ros_ray_sensor.so">
                 <ros>
-                    <namespace>KapiBara</namespace>
+                    <namespace>$(arg robot_name)</namespace>
                     <remapping>~/out:=${sensor_name}</remapping>
                 </ros>
                 <output_type>sensor_msgs/LaserScan</output_type>
                 <radiation_type>infrared</radiation_type>
-                <frame_name>${sensor_name}_laser</frame_name>
+                <frame_name>/$(arg robot_name)/${sensor_name}_laser</frame_name>
             </plugin>
         </sensor>

File: description/lasers_joints.xacro (robot description, xacro)
@@ -2,10 +2,10 @@
 <robot xmlns:xacro="http://www.ros.org/wiki/xacro">
     <!-- FRONT LEFT DISTANCE SENSOR -->
-    <joint name="front_left_laser_joint" type="fixed">
-        <parent link="base"/>
-        <child link="front_left_laser_link"/>
+    <joint name="/$(arg robot_name)/front_left_laser_joint" type="fixed">
+        <parent link="/$(arg robot_name)/base"/>
+        <child link="/$(arg robot_name)/front_left_laser_link"/>
         <origin xyz="-0.17 -0.04 0.04" rpy="0 0 ${pi}"/>
     </joint>
-    <link name="front_left_laser_link">
+    <link name="/$(arg robot_name)/front_left_laser_link">
         <visual>
             <geometry>
@@ -16,10 +16,10 @@
     </link>
     <!-- FRONT RIGHT DISTANCE SENSOR -->
-    <joint name="front_right_laser_joint" type="fixed">
-        <parent link="base"/>
-        <child link="front_right_laser_link"/>
+    <joint name="/$(arg robot_name)/front_right_laser_joint" type="fixed">
+        <parent link="/$(arg robot_name)/base"/>
+        <child link="/$(arg robot_name)/front_right_laser_link"/>
         <origin xyz="-0.17 0.04 0.04" rpy="0 0 ${pi}"/>
     </joint>
-    <link name="front_right_laser_link">
+    <link name="/$(arg robot_name)/front_right_laser_link">
         <visual>
             <geometry>
@@ -30,10 +30,10 @@
     </link>
     <!-- SIDE LEFT DISTANCE SENSOR -->
-    <joint name="side_left_laser_joint" type="fixed">
-        <parent link="base"/>
-        <child link="side_left_laser_link"/>
+    <joint name="/$(arg robot_name)/side_left_laser_joint" type="fixed">
+        <parent link="/$(arg robot_name)/base"/>
+        <child link="/$(arg robot_name)/side_left_laser_link"/>
         <origin xyz="-0.02 -0.06 0.04" rpy="0 0 ${-pi/2}"/>
     </joint>
-    <link name="side_left_laser_link">
+    <link name="/$(arg robot_name)/side_left_laser_link">
         <visual>
             <geometry>
@@ -44,10 +44,10 @@
     </link>
     <!-- SIDE RIGHT DISTANCE SENSOR -->
-    <joint name="side_right_laser_joint" type="fixed">
-        <parent link="base"/>
-        <child link="side_right_laser_link"/>
+    <joint name="/$(arg robot_name)/side_right_laser_joint" type="fixed">
+        <parent link="/$(arg robot_name)/base"/>
+        <child link="/$(arg robot_name)/side_right_laser_link"/>
         <origin xyz="-0.02 0.06 0.04" rpy="0 0 ${pi/2}"/>
     </joint>
-    <link name="side_right_laser_link">
+    <link name="/$(arg robot_name)/side_right_laser_link">
         <visual>
             <geometry>

File: description/robot_core.xacro (robot description, xacro)
@@ -15,13 +15,13 @@
     </material>
     <!-- BASE LINK -->
-    <link name="base_link">
+    <link name="/$(arg robot_name)/base_link">
     </link>
     <!-- CHASSIS LINK -->
-    <joint name="chassis_joint" type="fixed">
-        <parent link="base_link" />
-        <child link="chassis" />
+    <joint name="/$(arg robot_name)/chassis_joint" type="fixed">
+        <parent link="/$(arg robot_name)/base_link" />
+        <child link="/$(arg robot_name)/chassis" />
         <origin xyz="0 0 0" />
     </joint>
-    <link name="chassis">
+    <link name="/$(arg robot_name)/chassis">
         <visual>
             <origin xyz="0 0 0" />
@@ -32,14 +32,14 @@
         </visual>
     </link>
-    <gazebo reference="chassis">
+    <gazebo reference="/$(arg robot_name)/chassis">
         <material>Gazebo/Black</material>
     </gazebo>
     <!-- Base -->
-    <joint name="base_joint" type="fixed">
-        <parent link="chassis" />
-        <child link="base" />
+    <joint name="/$(arg robot_name)/base_joint" type="fixed">
+        <parent link="/$(arg robot_name)/chassis" />
+        <child link="/$(arg robot_name)/base" />
         <origin xyz="0.027 0 0.05" />
     </joint>
-    <link name="base">
+    <link name="/$(arg robot_name)/base">
         <visual>
             <origin xyz="0 0 0.05" />
@@ -59,5 +59,5 @@
         </xacro:inertial_box>
     </link>
-    <gazebo reference="base">
+    <gazebo reference="/$(arg robot_name)/base">
         <material>Gazebo/Orange</material>
         <sensor type="contact" name="contact_sensor">
@@ -69,5 +69,5 @@
             <plugin name="bumper_plugin_kapibara" filename="libgazebo_ros_bumper.so">
                 <alwaysOn>true</alwaysOn>
-                <frameName>base</frameName>
+                <frameName>/$(arg robot_name)/base</frameName>
                 <ros>
                 <remapping>bumper_states:=collision</remapping>
@@ -77,7 +77,7 @@
     </gazebo>
     <!-- LEFT WHEEL LINK -->
-    <joint name="wheel_left1_joint" type="continuous">
-        <parent link="chassis" />
-        <child link="left_wheel1" />
+    <joint name="/$(arg robot_name)/wheel_left1_joint" type="continuous">
+        <parent link="/$(arg robot_name)/chassis" />
+        <child link="/$(arg robot_name)/left_wheel1" />
         <axis xyz="0 0 1"/>
         <origin rpy="${-pi/2} 0 0" xyz="0.005 0.066 0.0135"/>
@@ -85,81 +85,81 @@
         <!-- <limit effort="10000" velocity="1000"/>  -->
     </joint>
-    <link name="left_wheel1">
-        <visual>
-            <origin xyz="0 0 0" />
-            <geometry>
-                <cylinder radius="0.024" length="0.044" />
-            </geometry>
-            <material name="white" />
-        </visual>
-        <collision>
-            <origin xyz="0 0 0" />
-            <geometry>
-                <cylinder radius="0.024" length="0.044" />
-            </geometry>
-        </collision>
-        <xacro:inertial_cylinder mass="0.1" radius="0.024" length="0.044">
-            <origin xyz="0 0 0" rpy="0 0 0" />
-        </xacro:inertial_cylinder>
-    </link>
-    <gazebo reference="left_wheel1">
-        <material>Gazebo/White</material>
-        <mu1 value="0.5"/>
-        <mu2 value="0.5"/>
-    </gazebo>
-    <joint name="wheel_left2_joint" type="continuous">
-        <parent link="chassis" />
-        <child link="left_wheel2" />
+    <link name="/$(arg robot_name)/left_wheel1">
+        <visual>
+            <origin xyz="0 0 0" />
+            <geometry>
+                <cylinder radius="0.024" length="0.044" />
+            </geometry>
+            <material name="white" />
+        </visual>
+        <collision>
+            <origin xyz="0 0 0" />
+            <geometry>
+                <cylinder radius="0.024" length="0.044" />
+            </geometry>
+        </collision>
+        <xacro:inertial_cylinder mass="0.1" radius="0.024" length="0.044">
+            <origin xyz="0 0 0" rpy="0 0 0" />
+        </xacro:inertial_cylinder>
+    </link>
+    <gazebo reference="/$(arg robot_name)/left_wheel1">
+        <material>Gazebo/White</material>
+        <mu1 value="0.5"/>
+        <mu2 value="0.5"/>
+    </gazebo>
+    <joint name="/$(arg robot_name)/wheel_left2_joint" type="continuous">
+        <parent link="/$(arg robot_name)/chassis" />
+        <child link="/$(arg robot_name)/left_wheel2" />
         <axis xyz="0 0 1"/>
         <origin rpy="${-pi/2} 0 0" xyz="0.065 0.066 0.0135"/>
     </joint>
-    <link name="left_wheel2">
-        <visual>
-            <origin xyz="0 0 0" />
-            <geometry>
-                <cylinder radius="0.024" length="0.044" />
-            </geometry>
-            <material name="white" />
-        </visual>
-        <collision>
-            <origin xyz="0 0 0" />
-            <geometry>
-                <cylinder radius="0.024" length="0.044" />
-            </geometry>
-        </collision>
-        <xacro:inertial_cylinder mass="0.1" radius="0.024" length="0.044">
-            <origin xyz="0 0 0" rpy="0 0 0" />
-        </xacro:inertial_cylinder>
-    </link>
-    <gazebo reference="left_wheel2">
-        <material>Gazebo/White</material>
-        <mu1 value="0.5"/>
-        <mu2 value="0.5"/>
-    </gazebo>
-    <joint name="wheel_left3_joint" type="continuous">
-        <parent link="chassis" />
-        <child link="left_wheel3" />
+    <link name="/$(arg robot_name)/left_wheel2">
+        <visual>
+            <origin xyz="0 0 0" />
+            <geometry>
+                <cylinder radius="0.024" length="0.044" />
+            </geometry>
+            <material name="white" />
+        </visual>
+        <collision>
+            <origin xyz="0 0 0" />
+            <geometry>
+                <cylinder radius="0.024" length="0.044" />
+            </geometry>
+        </collision>
+        <xacro:inertial_cylinder mass="0.1" radius="0.024" length="0.044">
+            <origin xyz="0 0 0" rpy="0 0 0" />
+        </xacro:inertial_cylinder>
+    </link>
+    <gazebo reference="/$(arg robot_name)/left_wheel2">
+        <material>Gazebo/White</material>
+        <mu1 value="0.5"/>
+        <mu2 value="0.5"/>
+    </gazebo>
+    <joint name="/$(arg robot_name)/wheel_left3_joint" type="continuous">
+        <parent link="/$(arg robot_name)/chassis" />
+        <child link="/$(arg robot_name)/left_wheel3" />
         <axis xyz="0 0 1"/>
         <origin rpy="${-pi/2} 0 0" xyz="-0.055 0.066 0.0135"/>
     </joint>
-    <link name="left_wheel3">
-        <visual>
-            <origin xyz="0 0 0" />
-            <geometry>
-                <cylinder radius="0.024" length="0.044" />
-            </geometry>
-            <material name="white" />
-        </visual>
-        <collision>
-            <origin xyz="0 0 0" />
-            <geometry>
-                <cylinder radius="0.024" length="0.044" />
-            </geometry>
-        </collision>
-        <xacro:inertial_cylinder mass="0.1" radius="0.024" length="0.044">
-            <origin xyz="0 0 0" rpy="0 0 0" />
-        </xacro:inertial_cylinder>
-    </link>
-    <gazebo reference="left_wheel3">
+    <link name="/$(arg robot_name)/left_wheel3">
+        <visual>
+            <origin xyz="0 0 0" />
+            <geometry>
+                <cylinder radius="0.024" length="0.044" />
+            </geometry>
+            <material name="white" />
+        </visual>
+        <collision>
+            <origin xyz="0 0 0" />
+            <geometry>
+                <cylinder radius="0.024" length="0.044" />
+            </geometry>
+        </collision>
+        <xacro:inertial_cylinder mass="0.1" radius="0.024" length="0.044">
+            <origin xyz="0 0 0" rpy="0 0 0" />
+        </xacro:inertial_cylinder>
+    </link>
+    <gazebo reference="/$(arg robot_name)/left_wheel3">
         <material>Gazebo/White</material>
         <mu1 value="0.5"/>
@@ -167,7 +167,7 @@
     </gazebo>
     <!-- RIGHT WHEEL LINK -->
-    <joint name="wheel_right1_joint" type="continuous">
-        <parent link="chassis" />
-        <child link="right_wheel1" />
+    <joint name="/$(arg robot_name)/wheel_right1_joint" type="continuous">
+        <parent link="/$(arg robot_name)/chassis" />
+        <child link="/$(arg robot_name)/right_wheel1" />
         <axis xyz="0 0 1"/>
         <origin rpy="${-pi/2} 0 0" xyz="0.005 -0.066 0.0135"/>
@@ -175,81 +175,81 @@
         <!-- <limit effort="10000" velocity="1000"/>  -->
     </joint>
-    <link name="right_wheel1">
-        <visual>
-            <origin xyz="0 0 0" />
-            <geometry>
-                <cylinder radius="0.024" length="0.044" />
-            </geometry>
-            <material name="white" />
-        </visual>
-        <collision>
-            <origin xyz="0 0 0" />
-            <geometry>
-                <cylinder radius="0.024" length="0.044" />
-            </geometry>
-        </collision>
-        <xacro:inertial_cylinder mass="0.1" radius="0.024" length="0.044">
-            <origin xyz="0 0 0" rpy="0 0 0" />
-        </xacro:inertial_cylinder>
-    </link>
-    <gazebo reference="right_wheel1">
-        <material>Gazebo/White</material>
-        <mu1 value="0.5"/>
-        <mu2 value="0.5"/>
-    </gazebo>
-    <joint name="wheel_right2_joint" type="continuous">
-        <parent link="chassis" />
-        <child link="right_wheel2" />
+    <link name="/$(arg robot_name)/right_wheel1">
+        <visual>
+            <origin xyz="0 0 0" />
+            <geometry>
+                <cylinder radius="0.024" length="0.044" />
+            </geometry>
+            <material name="white" />
+        </visual>
+        <collision>
+            <origin xyz="0 0 0" />
+            <geometry>
+                <cylinder radius="0.024" length="0.044" />
+            </geometry>
+        </collision>
+        <xacro:inertial_cylinder mass="0.1" radius="0.024" length="0.044">
+            <origin xyz="0 0 0" rpy="0 0 0" />
+        </xacro:inertial_cylinder>
+    </link>
+    <gazebo reference="/$(arg robot_name)/right_wheel1">
+        <material>Gazebo/White</material>
+        <mu1 value="0.5"/>
+        <mu2 value="0.5"/>
+    </gazebo>
+    <joint name="/$(arg robot_name)/wheel_right2_joint" type="continuous">
+        <parent link="/$(arg robot_name)/chassis" />
+        <child link="/$(arg robot_name)/right_wheel2" />
         <axis xyz="0 0 1"/>
         <origin rpy="${-pi/2} 0 0" xyz="0.065 -0.066 0.0135"/>
     </joint>
-    <link name="right_wheel2">
-        <visual>
-            <origin xyz="0 0 0" />
-            <geometry>
-                <cylinder radius="0.024" length="0.044" />
-            </geometry>
-            <material name="white" />
-        </visual>
-        <collision>
-            <origin xyz="0 0 0" />
-            <geometry>
-                <cylinder radius="0.024" length="0.044" />
-            </geometry>
-        </collision>
-        <xacro:inertial_cylinder mass="0.1" radius="0.024" length="0.044">
-            <origin xyz="0 0 0" rpy="0 0 0" />
-        </xacro:inertial_cylinder>
-    </link>
-    <gazebo reference="right_wheel2">
-        <material>Gazebo/White</material>
-        <mu1 value="0.5"/>
-        <mu2 value="0.5"/>
-    </gazebo>
-    <joint name="wheel_right3_joint" type="continuous">
-        <parent link="chassis" />
-        <child link="right_wheel3" />
+    <link name="/$(arg robot_name)/right_wheel2">
+        <visual>
+            <origin xyz="0 0 0" />
+            <geometry>
+                <cylinder radius="0.024" length="0.044" />
+            </geometry>
+            <material name="white" />
+        </visual>
+        <collision>
+            <origin xyz="0 0 0" />
+            <geometry>
+                <cylinder radius="0.024" length="0.044" />
+            </geometry>
+        </collision>
+        <xacro:inertial_cylinder mass="0.1" radius="0.024" length="0.044">
+            <origin xyz="0 0 0" rpy="0 0 0" />
+        </xacro:inertial_cylinder>
+    </link>
+    <gazebo reference="/$(arg robot_name)/right_wheel2">
+        <material>Gazebo/White</material>
+        <mu1 value="0.5"/>
+        <mu2 value="0.5"/>
+    </gazebo>
+    <joint name="/$(arg robot_name)/wheel_right3_joint" type="continuous">
+        <parent link="/$(arg robot_name)/chassis" />
+        <child link="/$(arg robot_name)/right_wheel3" />
         <axis xyz="0 0 1"/>
         <origin rpy="${-pi/2} 0 0" xyz="-0.055 -0.066 0.0135"/>
     </joint>
-    <link name="right_wheel3">
-        <visual>
-            <origin xyz="0 0 0" />
-            <geometry>
-                <cylinder radius="0.024" length="0.044" />
-            </geometry>
-            <material name="white" />
-        </visual>
-        <collision>
-            <origin xyz="0 0 0" />
-            <geometry>
-                <cylinder radius="0.024" length="0.044" />
-            </geometry>
-        </collision>
-        <xacro:inertial_cylinder mass="0.1" radius="0.024" length="0.044">
-            <origin xyz="0 0 0" rpy="0 0 0" />
-        </xacro:inertial_cylinder>
-    </link>
-    <gazebo reference="right_wheel3">
+    <link name="/$(arg robot_name)/right_wheel3">
+        <visual>
+            <origin xyz="0 0 0" />
+            <geometry>
+                <cylinder radius="0.024" length="0.044" />
+            </geometry>
+            <material name="white" />
+        </visual>
+        <collision>
+            <origin xyz="0 0 0" />
+            <geometry>
+                <cylinder radius="0.024" length="0.044" />
+            </geometry>
+        </collision>
+        <xacro:inertial_cylinder mass="0.1" radius="0.024" length="0.044">
+            <origin xyz="0 0 0" rpy="0 0 0" />
+        </xacro:inertial_cylinder>
+    </link>
+    <gazebo reference="/$(arg robot_name)/right_wheel3">
         <material>Gazebo/White</material>
         <mu1 value="0.5"/>
@@ -257,12 +257,12 @@
     </gazebo>
     <!-- EARS -->
-    <joint name="left_ear_joint" type="revolute">
-        <parent link="base" />
-        <child link="left_ear" />
+    <joint name="/$(arg robot_name)/left_ear_joint" type="revolute">
+        <parent link="/$(arg robot_name)/base" />
+        <child link="/$(arg robot_name)/left_ear" />
         <axis xyz="0 -1 0"/>
         <origin rpy="0 ${pi/2} 0" xyz="-0.09 0.075 0.09" />
         <limit effort="1" velocity="1" upper="${pi}" lower="0" />
     </joint>
-    <link name="left_ear">
+    <link name="/$(arg robot_name)/left_ear">
         <visual>
             <origin xyz="0 0 0" />
@@ -282,12 +282,12 @@
         </xacro:inertial_cylinder>
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