Commit message: I have fixed problem with TF

File: description/ros2_control.xacro (robot description, xacro)
@@ -5,6 +5,6 @@
             <hardware>
                 <plugin>vel_saltis_drive/VelSaltisDrive</plugin>
-                <param name="left_wheel_name">wheel_left1_joint</param>
-                <param name="right_wheel_name">wheel_right3_joint</param>
+                <param name="left_wheel_name">/$(arg robot_name)/wheel_left1_joint</param>
+                <param name="right_wheel_name">/$(arg robot_name)/wheel_right3_joint</param>
                 <!-- <param name="left_ear">left_ear_joint</param>
                 <param name="right_ear">right_ear_joint</param> -->
@@ -12,5 +12,5 @@
                 <param name="loop_rate">30</param>
             </hardware>
-            <joint name="wheel_left1_joint">
+            <joint name="/$(arg robot_name)/wheel_left1_joint">
                 <command_interface name="velocity">
                     <param name="min">-10</param>
@@ -20,5 +20,5 @@
                 <state_interface name="position" />
             </joint>
-            <joint name="wheel_right3_joint">
+            <joint name="/$(arg robot_name)/wheel_right3_joint">
                 <command_interface name="velocity">
                     <param name="min">-10</param>
@@ -46,9 +46,9 @@
             <hardware>
                 <plugin>vel_saltis_ears/VelSaltisEars</plugin>
-                <param name="left_ear_name">left_ear_joint</param>
-                <param name="right_ear_name">right_ear_joint</param>
+                <param name="left_ear_name">/$(arg robot_name)/left_ear_joint</param>
+                <param name="right_ear_name">/$(arg robot_name)/right_ear_joint</param>
                 <param name="loop_rate">30</param>
             </hardware>
-            <joint name="right_ear_joint">
+            <joint name="/$(arg robot_name)/right_ear_joint">
                 <command_interface name="position">
                     <param name="min">-10</param>
@@ -57,5 +57,5 @@
                 <state_interface name="position" />
             </joint>
-            <joint name="left_ear_joint">
+            <joint name="/$(arg robot_name)/left_ear_joint">
                 <command_interface name="position">
                     <param name="min">-10</param>
@@ -71,5 +71,5 @@
                 <plugin>gazebo_ros2_control/GazeboSystem</plugin>
             </hardware>
-            <joint name="wheel_left1_joint">
+            <joint name="/$(arg robot_name)/wheel_left1_joint">
                 <command_interface name="velocity">
                     <param name="min">-10</param>
@@ -79,5 +79,5 @@
                 <state_interface name="position" />
             </joint>
-            <joint name="wheel_right3_joint">
+            <joint name="/$(arg robot_name)/wheel_right3_joint">
                 <command_interface name="velocity">
                     <param name="min">-10</param>
@@ -87,5 +87,5 @@
                 <state_interface name="position" />
             </joint>
-            <joint name="right_ear_joint">
+            <joint name="/$(arg robot_name)/right_ear_joint">
                 <command_interface name="position">
                     <param name="min">-10</param>
@@ -94,5 +94,5 @@
                 <state_interface name="position" />
             </joint>
-            <joint name="left_ear_joint">
+            <joint name="/$(arg robot_name)/left_ear_joint">
                 <command_interface name="position">
                     <param name="min">-10</param>
@@ -106,9 +106,7 @@
         <plugin name="kapibara_gazebo_ros2_control" filename="libgazebo_ros2_control.so">
             <ros>
-                <namespace>KapiBara</namespace>
-                <remapping>/tf:=/KapiBara/tf</remapping>
-                <remapping>/tf_static:=/KapiBara/tf_static</remapping>
+                <namespace>$(arg robot_name)</namespace>
             </ros>
-            <robot_param_node>/KapiBara/robot_state_publisher</robot_param_node>
+            <robot_param_node>/$(arg robot_name)/robot_state_publisher</robot_param_node>
             <parameters>$(find kapibara)/config/my_controllers.yaml</parameters>
             <parameters>$(find kapibara)/config/my_controllers_sim.yaml</parameters>
